Commit message: Complete autonomous patrol control loop

File: src/robot_description/urdf/robot.urdf (robot description, URDF)
Before this commit: robot indoor_robot, 1 links, 0 joints
Links:
- added link base_footprint
- added link left_wheel; visual cylinder length=0.05 radius=0.10
- added link lidar_link; visual cylinder length=0.07 radius=0.06
- added link right_wheel; visual cylinder length=0.05 radius=0.10
- link base_link: mass 20 -> 20.0; geometry collision box size=0.60 0.40 0.20; visual box size=0.60 0.40 0.20
Joints:
- added joint base_footprint_joint: type fixed, parent base_footprint, child base_link
- added joint left_wheel_joint: type fixed, parent base_link, child left_wheel, origin xyz=0 0.225 0.10
- added joint lidar_joint: type fixed, parent base_link, child lidar_link, origin xyz=0.16 0 0.22
- added joint right_wheel_joint: type fixed, parent base_link, child right_wheel, origin xyz=0 -0.225 0.10
